File: Hardware/KiCAD files/Senior deisng mainboard32826 backup/motor_controls.kicad_sch (KiCad schematic)
At the start: 90 parts, among them J1 Conn_01x08, J11 Conn_01x08, J12 Conn_01x08, J16 JST_SMD_1.0mm_Vertical, J17 JST_SMD_1.0mm_Vertical, J2 Conn_01x08, J29 JST_SMD_1.0mm_Vertical, J4 JST_SMD_1.0mm_Vertical, J5 PINHD_1x8_Male, J9 PINHD_1x8_Male, U1 DRV8825PWPR, U10 DRV8825PWPR, U4 DRV8825PWPR, U5 DRV8825PWPR, U8 DRV8825PWPR, U9 DRV8825PWPR

Commit message: swapping connectors and rewiring through the project.
we verified connections with the ender3. a few placeholders replaced.
Parts:
- removed C19, C27, C34, C35, C42, C43, C47: 0.1uF, PCM_SparkFun-Capacitor:C_0603_1608Metric, symbol PCM_SparkFun-Capacitor:0.1uF_0603_100V_10%
- removed C2, C29, C37, C45: 10nF, PCM_SparkFun-Capacitor:C_0603_1608Metric, symbol PCM_SparkFun-Capacitor:10nF_0603_50V_10%
- removed C28, C36, C44, C5: 470nF, PCM_SparkFun-Capacitor:C_0402_1005Metric, symbol PCM_SparkFun-Capacitor:470nF_0402_25V_10%
- removed C30, C38, C4, C46, C7, C8: 0.1uF, PCM_SparkFun-Capacitor:C_0603_1608Metric, symbol PCM_SparkFun-Capacitor:0.1uF_0603_25V_20%
- removed C32, C40, C48: 100uF_50V, Capacitor_THT:CP_Radial_D8.0mm_P3.50mm, symbol PCM_SL_Capacitors:100uF_50V
- removed C33, C41, C6: 4.7uF, PCM_SparkFun-Capacitor:C_0603_1608Metric, symbol PCM_SparkFun-Capacitor:4.7uF_0603_35V_20%
- removed J1, J2: Conn_01x08, PCM_SparkFun-Connector:1x08_P2.54mm, symbol PCM_SparkFun-Connector:Conn_01x08_P2.54mm
- removed J16, J17, J29, J4: JST_SMD_1.0mm_Vertical, PCM_SparkFun-Connector:JST_1x04_P1.0mm_Vertical_SMD, symbol PCM_SparkFun-Connector:Conn_01x04_JST_P1.0mm_Vertical_SMD
- removed R19: .2 ohm, symbol PCM_Resistor_AKL:R_Generic
- removed R20, R26, R31, R6: 1.5k, PCM_SparkFun-Resistor:R_0603_1608Metric, symbol PCM_SparkFun-Resistor:1.5k_0603
- removed R22, R27, R32: 1_Mohm, symbol PCM_Resistor_AKL:R_Generic
- removed R23, R28, R33, R5: 10k Linear, PCM_SparkFun-Resistor:Bourns-PDB18, symbol PCM_SparkFun-Resistor:Trimpot_10k_RA_PTH
- removed R24, R29, R34, R9: 10k, PCM_SparkFun-Resistor:R_0603_1608Metric, symbol PCM_SparkFun-Resistor:10k_0603
- removed U1: DRV8825PWPR, PWP28_5P18X3P1, symbol DRV8825PRPR driver chip:DRV8825PWPR
- added C13, C14, C15, C32, C36, C40, C44: 0.1uF, PCM_SparkFun-Capacitor:C_0603_1608Metric, symbol PCM_SparkFun-Capacitor:0.1uF_0603_100V_10%
- added C19, C37, C45: 100uF_50V, Capacitor_THT:CP_Radial_D8.0mm_P3.50mm, symbol PCM_SL_Capacitors:100uF_50V
- added C27, C33, C41: 470nF, PCM_SparkFun-Capacitor:C_0402_1005Metric, symbol PCM_SparkFun-Capacitor:470nF_0402_25V_10%
- added C28, C34, C42: 10nF, PCM_SparkFun-Capacitor:C_0603_1608Metric, symbol PCM_SparkFun-Capacitor:10nF_0603_50V_10%
- added C29, C35, C43: 0.1uF, PCM_SparkFun-Capacitor:C_0603_1608Metric, symbol PCM_SparkFun-Capacitor:0.1uF_0603_25V_20%
- added C30, C38: 4.7uF, PCM_SparkFun-Capacitor:C_0603_1608Metric, symbol PCM_SparkFun-Capacitor:4.7uF_0603_35V_20%
- added J2, J4, J6, J7: Conn_01x06, PCM_SparkFun-Connector:1x06_P2.54mm, symbol PCM_SparkFun-Connector:Conn_01x06_P2.54mm
- added R19, R24, R29: 1.5k, PCM_SparkFun-Resistor:R_0603_1608Metric, symbol PCM_SparkFun-Resistor:1.5k_0603
- added R20: 1_Mohm, symbol PCM_Resistor_AKL:R_Generic
- added R21, R26, R31: 10k Linear, PCM_SparkFun-Resistor:Bourns-PDB18, symbol PCM_SparkFun-Resistor:Trimpot_10k_RA_PTH
- added R22, R27, R32: 10k, PCM_SparkFun-Resistor:R_0603_1608Metric, symbol PCM_SparkFun-Resistor:10k_0603
- added R23, R28, R9: .2 ohm, symbol PCM_Resistor_AKL:R_Generic
- C10, C11, C17, C18, C31, C39, C52, C53, C54: now not fitted
- R25, R30: value .2 ohm -> 1_Mohm
- U10, U4, U5, U8, U9: footprint PWP28_5P18X3P1 -> (none)
Connections:
- net DRIVER_1_STEP is gone; now on net DRIVER_0_STEP: U8.22 (STEP)
- net DRIVER_2_STEP is gone; now on net DRIVER_0_STEP: U10.22 (STEP), U9.22 (STEP)
- net +24V: now also R25.1, R30.1, C13.1, C14.1, C15.1, C19.1, C29.1, C30.1, C32.1, C35.1, C36.1, C37.1, C38.1, C40.1, C43.1, C44.1, C45.1, R20.1
- net +3V3: now also C27.1, C33.1, C41.1, R21.3, R26.3, R31.3
- net A1: now also J2.6 (Pin_6), J4.6 (Pin_6), J6.6 (Pin_6), J7.6 (Pin_6)
- net A2: now also J2.3 (Pin_3), J4.3 (Pin_3), J6.3 (Pin_3), J7.3 (Pin_3)
- net B1: now also J2.4 (Pin_4), J4.4 (Pin_4), J6.4 (Pin_4), J7.4 (Pin_4)
- net B2: now also J2.1 (Pin_1), J4.1 (Pin_1), J6.1 (Pin_1), J7.1 (Pin_1)
- net GND: now also C13.2, C14.2, C15.2, C19.2, C27.2, C30.2, C32.2, C33.2, C36.2, C37.2, C38.2, C40.2, C41.2, C44.2, C45.2, R21.1, R23.1, R26.1, R28.1, R31.1, R9.1; no longer R25.1, R30.1
- net N_FAULT: now also R19.2, R22.1, R24.2, R27.1, R29.2, R32.1
- net SLP: now also R22.2, R27.2, R32.2
- net at U9.1 (CP1): now also C34.1
- net at U9.2 (CP2): now also C34.2
- net at U9.12 (AVREF), U9.13 (BVREF): now also R26.2
- net at U9.18 (NFAULT): now also R24.1
- net at U9.3 (VCP): now also R25.2, C35.2
- net at U9.6 (ISENA), U9.9 (ISENB): now also R23.2; no longer R25.2
- net at U10.12 (AVREF), U10.13 (BVREF): now also R31.2
- net at U8.3 (VCP): now also C29.2, R20.2
- net at U10.3 (VCP): now also R30.2, C43.2
- net at U10.1 (CP1): now also C42.1
- net at U10.18 (NFAULT): now also R29.1
- net at U10.2 (CP2): now also C42.2
- net at U10.6 (ISENA), U10.9 (ISENB): now also R28.2; no longer R30.2
- net at U8.18 (NFAULT): now also R19.1
- net at U8.6 (ISENA), U8.9 (ISENB): now also R9.2
- net at U8.1 (CP1): now also C28.1
- net at U8.2 (CP2): now also C28.2
- net at U8.12 (AVREF), U8.13 (BVREF): now also R21.2
- no-connect marks 24 -> 28
Other:
- note added: "DRV8825 1.1 D0"
- note added: "DRV8825 1.1 D02"
- note added: "DRV8825 1.1 D03 Extruder"
- note added: "DRV8825 1.1 D1"
- note added: "verify that board phase wiring is switched to match jst connector"
- note removed: "DRV8825 1.0 D0"
- note removed: "DRV8825 1.0 D02"
- note removed: "DRV8825 1.0 D03 Extruder"
- note removed: "DRV8825 1.0 D1"
- note removed: "DRV8825 1.0 Standalone"
- note removed: "NEED TO RE-IMPLEMENT EXRUDER DRIVER, individual control necessary"
- note removed: "NoteMeausure impedance of the lines in layout ISA and ISB are .10 ohm"
- note removed: "This is designed as a standalone, J1 and J2 removed for mainboard."
- note removed: "previous design for reference"

Commit message: New project made to reflect layouts
New project files made in order to generate accurate layouts and create neatness.
Connections:
- net SLP: now also J5.3, U5.17 (NSLEEP)
Changed lines of the file:
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@@
 	)
 	(junction
+		(at 31.75 66.04)
+		(diameter 0)
+		(color 0 0 0 0)
+	)
+	(junction
 		(at 304.8 177.8)
 		(diameter 0)
@@
 	(wire
 		(pts
-			(xy 478.79 69.85) (xy 478.79 78.74)
+			(xy 478.79 69.85) (xy 478.79 83.82)
 		)
 		(stroke
@@
 	(wire
 		(pts
-			(xy 453.39 77.47) (xy 473.71 77.47)
-		)
-		(stroke
-			(width 0)
-			(type default)
-		)
-	)
-	(wire
-		(pts
 			(xy 210.82 57.15) (xy 210.82 50.8)
 		)
@@
 	(wire
 		(pts
-			(xy 483.87 76.2) (xy 483.87 78.74)
-		)
-		(stroke
-			(width 0)
-			(type default)
-		)
-	)
-	(wire
-		(pts
 			(xy 156.21 34.29) (xy 162.56 34.29)
 		)
@@
 	(wire
 		(pts
-			(xy 482.6 78.74) (xy 482.6 83.82)
-		)
-		(stroke
-			(width 0)
-			(type default)
-		)
-	)
-	(wire
-		(pts
 			(xy 288.29 74.93) (xy 293.37 74.93)
 		)
@@
 	(wire
 		(pts
-			(xy 478.79 78.74) (xy 482.6 78.74)
+			(xy 478.79 83.82) (xy 486.41 83.82)
 		)
 		(stroke
@@
 	(wire
 		(pts
-			(xy 453.39 74.93) (xy 477.52 74.93)
+			(xy 457.2 73.66) (xy 457.2 77.47)
+		)
+		(stroke
+			(width 0)
+			(type default)
+		)
+	)
+	(wire
+		(pts
+			(xy 453.39 74.93) (xy 483.87 74.93)
 		)
 		(stroke
@@
 	(wire
 		(pts
-			(xy 477.52 74.93) (xy 477.52 81.28)
+			(xy 483.87 74.93) (xy 483.87 76.2)
 		)
 		(stroke
@@
 	(wire
 		(pts
+			(xy 31.75 57.15) (xy 31.75 66.04)
+		)
+		(stroke
+			(width 0)
+			(type default)
+		)
+	)
+	(wire
+		(pts
 			(xy 133.35 176.53) (xy 135.89 176.53)
 		)
@@
 	(wire
 		(pts
-			(xy 483.87 78.74) (xy 486.41 78.74)
-		)
-		(stroke
-			(width 0)
-			(type default)
-		)
-	)
-	(wire
-		(pts
 			(xy 123.19 57.15) (xy 124.46 57.15)
 		)
@@
 	(wire
 		(pts
+			(xy 457.2 77.47) (xy 453.39 77.47)
+		)
+		(stroke
+			(width 0)
+			(type default)
+		)
+	)
+	(wire
+		(pts
 			(xy 137.16 34.29) (xy 144.78 34.29)
 		)
@@
 	(wire
 		(pts
-			(xy 467.36 82.55) (xy 467.36 76.2)
+			(xy 467.36 82.55) (xy 467.36 78.74)
 		)
 		(stroke
@@
 	(wire
 		(pts
-			(xy 485.14 81.28) (xy 485.14 76.2)
-		)
-		(stroke
-			(width 0)
-			(type default)
-		)
-	)
-	(wire
-		(pts
-			(xy 473.71 77.47) (xy 473.71 73.66)
-		)
-		(stroke
-			(width 0)
-			(type default)
-		)
-	)
-	(wire
-		(pts
 			(xy 382.27 69.85) (xy 373.38 69.85)
 		)
@@
 	(wire
 		(pts
-			(xy 22.86 66.04) (xy 39.37 66.04)
+			(xy 22.86 66.04) (xy 31.75 66.04)
 		)
 		(stroke
@@
 	(wire
 		(pts
-			(xy 473.71 73.66) (xy 485.14 73.66)
+			(xy 457.2 73.66) (xy 485.14 73.66)
+		)
+		(stroke
+			(width 0)
+			(type default)
+		)
+	)
+	(wire
+		(pts
+			(xy 31.75 66.04) (xy 39.37 66.04)
 		)
 		(stroke
@@
 	(wire
 		(pts
-			(xy 485.14 76.2) (xy 486.41 76.2)
+			(xy 483.87 76.2) (xy 486.41 76.2)
 		)
 		(stroke
@@
 	(wire
 		(pts
-			(xy 482.6 83.82) (xy 486.41 83.82)
-		)
-		(stroke
-			(width 0)
-			(type default)
-		)
-	)
-	(wire
-		(pts
 			(xy 25.4 220.98) (xy 43.18 220.98)
 		)
@@
 	(wire
 		(pts
-			(xy 477.52 81.28) (xy 485.14 81.28)
-		)
-		(stroke
-			(width 0)
-			(type default)
-		)
-	)
-	(wire
-		(pts
 			(xy 476.25 86.36) (xy 480.06 86.36)
 		)
@@
 	(wire
 		(pts
-			(xy 467.36 76.2) (xy 483.87 76.2)
+			(xy 467.36 78.74) (xy 486.41 78.74)
 		)
 		(stroke
@@
 		)
 	)
-	(label "B1"
-		(at 467.36 76.2 180)
-		(effects
-			(font
-				(size 0.508 0.508)
-			)
-			(justify right bottom)
-		)
-	)
 	(label "Set Home"
 		(at 538.48 313.69 180)
@@
 		)
 	)
-	(label "B2"
-		(at 473.71 73.66 180)
-		(effects
-			(font
-				(size 0.508 0.508)
-			)
-			(justify right bottom)
-		)
-	)
 	(label "B1"
 		(at 135.89 213.36 180)
@@
 		)
 	)
-	(label "A1"
-		(at 478.79 78.74 180)
+	(label "B2"
+		(at 485.14 71.12 180)
 		(effects
 			(font
@@
 	)
 	(label "A2"
-		(at 477.52 81.28 180)
+		(at 483.87 76.2 180)
+		(effects
+			(font
+				(size 0.508 0.508)
+			)
+			(justify right bottom)
+		)
+	)
+	(label "A1"
+		(at 483.87 83.82 180)
 		(effects
 			(font
@@
 		)
 	)
+	(label "B1"
+		(at 481.33 78.74 180)
+		(effects
+			(font
+				(size 0.508 0.508)
+			)
+			(justify right bottom)
+		)
+	)
 	(label "A2"
 		(at 146.05 218.44 180)
@@
 	)
 	(global_label "SLP"
-		(shape input)
+		(shape output)
 		(at 163.83 59.69 0)
 		(fields_autoplaced yes)
@@
 			)
 		)
+	)
+	(global_label "SLP"
+		(shape input)
+		(at 31.75 57.15 90)
+		(fields_autoplaced yes)
+		(effects
+			(font
+				(size 1.27 1.27)
+			)
+			(justify left)
+		)
+		(property "Intersheetrefs" "${INTERSHEET_REFS}"
+			(at 31.75 50.6572 90)
+			(hide yes)
+			(show_name no)
+			(do_not_autoplace no)
+			(effects
+				(font
+					(size 1.27 1.27)
+				)
+				(justify left)
+			)
+		)
