File: Hardware/KiCAD files/Mainboard layout/Mainboard layout.kicad_sch (KiCad schematic)
At the start: 67 parts, among them J1 MSD-1-A, J10 Conn_01x02, J11 Conn_01x04, J12 JST_06, J13 Conn_01x08, J17 PINHD_1x8_Male, J18 PINHD_1x8_Male, J19 PINHD_1x8_Male, J2 Screw_Terminal_2_P5.00mm, J20 PINHD_1x8_Male, J22 PINHD_1x8_Male, J23 PINHD_1x8_Male, J24 PINHD_1x8_Male, J25 Conn_01x04, J26 Conn_01x04, J27 Conn_01x04, J28 PINHD_1x8_Male, J3 Screw_Terminal_2_P3.50mm, J30 USB-A1VSB6, J31 JST_03, J34 JST_03, J35 JST_03, J36 JST_03, J37 JST_03, J38 JST_03, J4 JST_06, J5 Conn_01x04, J6 JST_06, J7 JST_06, J8 Conn_01x06, J9 Conn_01x10, Q1 BS170, Q2 2DD1664, SW8 Push_Button, SW9 Push_Button, U12 ESP32-S3-WROOM-1, U3 PCA9534PW, U5 PCA9534PW

Commit message: general progress and adjustments
new footprint for pi reg inductor, var reg checked concurred with current part and value. re footprinted motor driver. started swapping head. adjusted some device footprints.
Parts:
- removed C1: 1nF_Ceramic, Capacitor_THT:C_Disc_D5.0mm_W2.5mm_P2.50mm, symbol PCM_SL_Capacitors:1nF_Ceramic
- removed R39: 10k, Resistor_THT:R_Axial_DIN0207_L6.3mm_D2.5mm_P10.16mm_Horizontal, symbol PCM_SL_Resistors:10k
- removed R54: 10k, PCM_SparkFun-Resistor:R_0603_1608Metric, symbol PCM_SparkFun-Resistor:10k_0603
- removed R6: 1M, PCM_SparkFun-Resistor:R_0603_1608Metric, symbol PCM_SparkFun-Resistor:1M_0603
- added C6, C7: 0.1uF, PCM_SparkFun-Capacitor:C_0603_1608Metric, symbol PCM_SparkFun-Capacitor:0.1uF_0603_25V_20%
- added C8: 1.0uF, PCM_SparkFun-Capacitor:C_0805_2012Metric, symbol PCM_SparkFun-Capacitor:1.0uF_0805_25V_10%
- added C9: 4.7uF, PCM_SparkFun-Capacitor:C_0603_1608Metric, symbol PCM_SparkFun-Capacitor:4.7uF_0603_35V_20%
- added D1: SP0502BAJT, PCM_Package_TO_SOT_SMD_AKL:SOT-323_SC-70, symbol PCM_Diode_TVS_AKL:SP0502BAJT
- added D10, D11: SP0503BAHT, PCM_Package_TO_SOT_SMD_AKL:SOT-143, symbol PCM_Diode_TVS_AKL:SP0503BAHT
- added J32: USB-A1VSB6, Connector_USB:USB_A_Kycon_KUSBX-AS1N-B_Horizontal, symbol USB-A1VSB6:USB-A1VSB6
- added R41, R6, R8: 10k, Resistor_THT:R_Axial_DIN0207_L6.3mm_D2.5mm_P10.16mm_Horizontal, symbol PCM_SL_Resistors:10k
- added R57: 10k, PCM_SparkFun-Resistor:R_0603_1608Metric, symbol PCM_SparkFun-Resistor:10k_0603
- added SW1, SW2, SW3, SW4: 210-4MS, 4-pin DIP switch:DIP8_210-4_CTS, symbol 2026-04-21_02-24-22:210-4MS
- added U1: CP2102-GM, CP2102:QFN28_5X5_SIL, symbol 2026-04-20_20-31-56:CP2102-GM
- J1: footprint CONN9_MSD-1_CUD -> Connector_Card:SD_Hirose_DM1AA_SF_PEJ82
- R40: value 100k -> 10k
Connections:
- net +5V: now also J3.2, C7.1, C8.1, U1.7 (REGIN)
- net +5V_HIGHPW: now also D11.2 (L1), J32.1 (VUSB); no longer J30.1 (VUSB)
- net 3.3V_in1: now also Q1.2 (G), U3.7 (IO3), R41.1; no longer Q1.3 (S), U12.15 (GPIO3/TOUCH3/ADC1_CH2)
- net AXIS_X_ENDSTOP: now also U5.9 (IO4); no longer U12.6 (GPIO6/TOUCH6/ADC1_CH5)
- net AXIS_Y_ENDSTOP: now also U5.10 (IO5); no longer U12.5 (GPIO5/TOUCH5/ADC1_CH4)
- net GND: now also J30.4 (GND), J30.S1 (SHIELD), J30.S2 (SHIELD__1), Q1.3 (S), C6.2, C7.2, C8.2, C9.2, D1.3 (A), D10.1 (VN), D11.1 (VN), J32.4 (GND), J32.S1 (SHIELD), J32.S2 (SHIELD__1), R6.2, R8.1, U1.29 (EPAD), U1.3 (GND); no longer J3.2
- net MODE_0_GPIOE: now also SW1.8; no longer U3.10 (IO5)
- net MODE_1_GPIOE: now also SW1.7; no longer U3.9 (IO4)
- net MODE_2_GPIOE: now also SW1.6; no longer U3.7 (IO3)
- net RX: now also D1.1 (K1), U1.25 (RXD)
- net TX: now also D1.2 (K2), U1.26 (TXD)
- net nSLP: now also U3.6 (IO2); no longer U12.16 (GPIO46)
- net 3.3V: now reaches U5.16 (VDD)
- net 3.3V: now also C16.1, C2.1, C23.1, J1.4 (VDD), J13.3 (Pin_3), J26.1 (Pin_1), J31.1, J34.1, J35.3, J36.3, J37.3, J38.3, J5.1 (Pin_1), J9.1 (Pin_1), J9.8 (Pin_8), R36.1, R48.1, R49.2, R5.1, R50.2, R52.2, R53.2, R55.1, R56.2, U12.2 (3V3), U3.16 (VDD), C6.1, C9.1, R41.2, R57.1, SW1.1, SW1.2, SW1.3, SW1.4, SW2.1, SW2.2, SW2.3, SW2.4, SW3.1, SW3.2, SW3.3, SW3.4, SW4.1, SW4.2, SW4.3, SW4.4, U1.6 (VDD)
- net DTR: now reaches U12.24 (GPIO47/SPICLK_P/SUBSPICLK_P_DIFF)
- net DTR: now also U1.28 (DTR)
- net RST: now reaches U12.25 (GPIO48/SPICLK_N/SUBSPICLK_N_DIFF)
- net RST: now also U1.9 (*RST)
- net IO_Interupter2: now reaches U12.32 (MTCK/GPIO39/CLK_OUT3/SUBSPICS1)
- net IO_Interupter2: now also U5.13 (~{INT}), R57.2
- net DSR: now reaches U12.33 (MTDO/GPIO40/CLK_OUT2)
- net DSR: now also U1.27 (DSR)
- removed net +3.3V: C16.1, C2.1, C23.1, J1.4 (VDD), J13.3 (Pin_3), J26.1 (Pin_1), J31.1, J34.1, J35.3, J36.3, J37.3, J38.3, J5.1 (Pin_1), J9.1 (Pin_1), J9.8 (Pin_8), Q1.2 (G), R36.1, R48.1, R49.2, R5.1, R50.2, R52.2, R53.2, R55.1, R56.2, U12.2 (3V3), U3.16 (VDD)
- net D+ renamed PI_D+
- net PI_D+: now also D11.4 (L3), J32.3 (D+); no longer J30.3 (D+)
- net D- renamed PI_D-
- net PI_D-: now also D11.3 (L2), J32.2 (D-); no longer J30.2 (D-)
- net IO_Interupter renamed IO_Interupter1
- net IO_Interupter1: no longer U5.13 (~{INT})
- removed net MODE_0_GPIO: J22.4, J23.4, J24.4, U3.4 (IO0)
- removed net MODE_1_GPIO: J22.3, J23.3, J24.3, U3.5 (IO1)
- removed net MODE_2_GPIO: J22.2, J23.2, J24.2, U3.6 (IO2)
- new net *Suspend: R6.1, U1.11 (*SUSPEND), U3.5 (IO1)
- new net CTS: U1.23 (CTS), U12.16 (GPIO46)
- new net DCD: U1.1 (DCD), U12.6 (GPIO6/TOUCH6/ADC1_CH5)
- new net MODE_0_GPIO0: J23.4, SW3.8
- new net MODE_0_GPIO1: J22.4, SW2.8
- new net MODE_0_GPIO2: J24.4, SW4.8
- new net MODE_1_GPIO0: J23.3, SW3.7
- new net MODE_1_GPIO1: J22.3, SW2.7
- new net MODE_1_GPIO2: J24.3, SW4.7
- new net MODE_2_GPIO0: J23.2, SW3.6
- new net MODE_2_GPIO1: J22.2, SW2.6
- new net MODE_2_GPIO2: J24.2, SW4.6
- new net Prog_D+: D10.4 (L3), J30.3 (D+), U1.4 (D+)
- new net Prog_D-: D10.3 (L2), J30.2 (D-), U1.5 (D-)
- new net RI: U1.2 (RI), U12.5 (GPIO5/TOUCH5/ADC1_CH4)
- new net RTS: U1.24 (RTS), U12.15 (GPIO3/TOUCH3/ADC1_CH2)
- new net Suspend: R8.2, U1.12 (SUSPEND), U3.4 (IO0)
- new net VBus: D10.2 (L1), J30.1 (VUSB), U1.8 (VBUS)
- no-connect marks 22 -> 32
Other:
- note added: "CHECK FOOTPRINT FOR LARGER VERSION"
- note added: "Check"
- note added: "Programmer_USB"
- note added: "RST - open drain output Regin - 5V in? CTS - Active low RTS - Active low DSR - Active Low DTR - Active Low DCD - Active Low RI - Active Low"
- note added: "TVS diode array or equivalent to SP0502BAHTG equivalent"
- note added: "USB_PI"
- note added: "Verify diodes"
- note removed: "USB"
- moved on the sheet: C23, J30, R56, U5

Commit message: general updates to the schematics and layouts
includes some backchecks tot he master schematic to be accurate for the paper
Other:
- note added: "CP2102"
- note added: "DIP SWITCHES"
- note added: "ENDSTOP INPUTS"
- note added: "FANS"
- note added: "HOTPLATE PERIPHERAL CONNECTIONS"
- note added: "MCU"
- note added: "MOTOR DRIVERS"
- note added: "REGULATORS 3.3V, 5V, 12V"
- note added: "SD CARD"
- note added: "STEP DISPERSAL"
- note removed: "CHECK FOOTPRINT FOR LARGER VERSION"
- note removed: "NEED TO VERIFY IF I CAN CHAIN THESE"
- note removed: "double check these values"
- note removed: "endstop inputs"
- note removed: "hotplate peripheral connections"
- moved on the sheet: C16, C2, C23, C3, C4, C6, C7, C8, C9, D1, D10, D11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
