File: Hardware/KiCAD files/Mainboard layout/Mainboard layout.kicad_sch (KiCad schematic)
At the start: 82 parts, among them J10 Conn_01x02, J11 Conn_01x04, J12 JST_06, J13 Conn_01x08, J14 Conn_01x08, J17 PINHD_1x8_Male, J18 PINHD_1x8_Male, J19 PINHD_1x8_Male, J2 Screw_Terminal_2_P5.00mm, J20 PINHD_1x8_Male, J22 PINHD_1x8_Male, J23 PINHD_1x8_Male, J24 PINHD_1x8_Male, J25 Conn_01x04, J26 Conn_01x04, J27 Conn_01x04, J28 PINHD_1x8_Male, J3 Screw_Terminal_2_P3.50mm, J30 USB-A1VSB6, J31 JST_03, J32 USB-A1VSB6, J34 JST_03, J35 JST_03, J36 JST_03, J37 JST_03, J38 JST_03, J4 JST_06, J5 Conn_01x04, J6 JST_06, J7 JST_06, J8 Conn_01x06, J9 Conn_01x10, Q1 BS170, Q2 2DD1664, SW1 210-4MS, SW2 210-4MS, SW3 210-4MS, SW4 210-4MS, SW8 Push_Button, SW9 Push_Button, U1 CP2102-GM, U12 ESP32-S3-WROOM-1, U2 PCA9534PW_118, U4 PCA9534PW_118

Commit message: Slight adjustments for EMI
trace changes primarily
Parts:
- added J15: Screw_Terminal_2_P5.00mm, TerminalBlock_Phoenix:TerminalBlock_Phoenix_PT-1,5-2-5.0-H_1x02_P5.00mm_Horizontal, symbol PCM_SL_Screw_Terminal:Screw_Terminal_2_P5.00mm
- added R9: 1k, Resistor_SMD:R_0805_2012Metric, symbol PCM_SL_Resistors:1k
- C16: footprint PCM_SparkFun-Capacitor:C_0603_1608Metric -> LED_SMD:LED_0805_2012Metric
- C23: footprint PCM_SparkFun-Capacitor:C_0603_1608Metric -> Capacitor_SMD:C_0805_2012Metric
- R52, R53: footprint PCM_SparkFun-Resistor:R_0603_1608Metric -> LED_SMD:LED_0805_2012Metric
- R55, R56, R57: footprint PCM_SparkFun-Resistor:R_0603_1608Metric -> Resistor_SMD:R_0805_2012Metric
- U2, U4: footprint PCA9534PW_118:SOP65P640X110-16N -> PCA9534PW:SOP65P640X110-16N
Connections:
- net Step is gone; now on net STEP: R50.1, U12.4 (GPIO4/TOUCH4/ADC1_CH3)
- net DRIVER_0_STEP: no longer J28.7, R107.1
- net STEPE: now reaches U4.4 (IO0)
- net STEPE: now also R9.2
- new net DRIVER_E_STEP: J28.7, R107.1, R9.1
- no-connect marks 33 -> 34
Other:
- note added: "IN CASE FOR SHIELDING"
- note removed: "Check"
- note removed: "change val"
- note removed: "rasberry pi connector"

Commit message: slight addition
includes some things that DR. weeks mentioned in class
Parts:
- added D2, D3: SP0503BAHT, PCM_Package_TO_SOT_SMD_AKL:SOT-143, symbol PCM_Diode_TVS_AKL:SP0503BAHT
Other:
- note added: "Pre-lim idea on muting backfeed onn 3.3V line"
Changed lines of the file:
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@@
 		)
 	)
+	(text "Pre-lim idea on muting backfeed onn 3.3V line\n"
+		(exclude_from_sim no)
+		(at 29.464 218.186 0)
+		(effects
+			(font
+				(size 1.27 1.27)
+			)
+		)
+	)
 	(text "ENDSTOP INPUTS"
 		(exclude_from_sim no)
@@
 	)
 	(symbol
+		(lib_id "PCM_Diode_TVS_AKL:SP0503BAHT")
+		(at 24.13 243.84 180)
+		(unit 1)
+		(body_style 1)
+		(exclude_from_sim no)
+		(in_bom yes)
+		(on_board yes)
+		(in_pos_files yes)
+		(dnp yes)
+		(fields_autoplaced yes)
+		(property "Reference" "D3"
+			(at 31.75 242.5699 0)
+			(show_name no)
+			(do_not_autoplace no)
+			(effects
+				(font
+					(size 1.27 1.27)
+				)
+				(justify right)
+			)
+		)
+		(property "Value" "SP0503BAHT"
+			(at 31.75 245.1099 0)
+			(show_name no)
+			(do_not_autoplace no)
+			(effects
+				(font
+					(size 1.27 1.27)
+				)
+				(justify right)
+			)
+		)
+		(property "Footprint" "PCM_Package_TO_SOT_SMD_AKL:SOT-143"
+			(at 24.13 243.84 0)
+			(hide yes)
+			(show_name no)
+			(do_not_autoplace no)
+			(effects
+				(font
+					(size 1.27 1.27)
+				)
+			)
+		)
+		(property "Datasheet" "https://www.tme.eu/Document/ca7ed7e840192927c2f50631891ac6c9/SP05xxBA.pdf"
+			(at 24.13 243.84 0)
+			(hide yes)
+			(show_name no)
+			(do_not_autoplace no)
+			(effects
+				(font
+					(size 1.27 1.27)
+				)
+			)
+		)
+		(property "Description" "SOT-143 TVS Diode array, 3xUnidirectional, 5.5V, Alternate KiCAD Library"
+			(at 24.13 243.84 0)
+			(hide yes)
+			(show_name no)
+			(do_not_autoplace no)
+			(effects
+				(font
+					(size 1.27 1.27)
+				)
+			)
+		)
+		(pin "1"
+		)
+		(pin "2"
+		)
+		(pin "4"
+		)
+		(pin "3"
+		)
+		(instances
+			(project "Mainboard layout"
+				(path "/322d2c9f-d9a6-40cc-b638-389f55be9478"
+					(reference "D3")
+					(unit 1)
+				)
+			)
+		)
+	)
+	(symbol
 		(lib_id "PCM_SparkFun-Connector:Conn_01x04_P2.54mm")
 		(at 417.83 341.63 270)
@@
 					(unit 1)
 				)
+			)
+		)
+	)
+	(symbol
+		(lib_id "PCM_Diode_TVS_AKL:SP0503BAHT")
+		(at 24.13 227.33 180)
+		(unit 1)
+		(body_style 1)
+		(exclude_from_sim no)
+		(in_bom yes)
+		(on_board yes)
+		(in_pos_files yes)
+		(dnp yes)
+		(fields_autoplaced yes)
+		(property "Reference" "D2"
+			(at 31.75 226.0599 0)
+			(show_name no)
+			(do_not_autoplace no)
+			(effects
+				(font
+					(size 1.27 1.27)
+				)
+				(justify right)
+			)
+		)
+		(property "Value" "SP0503BAHT"
+			(at 31.75 228.5999 0)
+			(show_name no)
+			(do_not_autoplace no)
+			(effects
+				(font
+					(size 1.27 1.27)
+				)
+				(justify right)
+			)
+		)
+		(property "Footprint" "PCM_Package_TO_SOT_SMD_AKL:SOT-143"
+			(at 24.13 227.33 0)
+			(hide yes)
+			(show_name no)
+			(do_not_autoplace no)
+			(effects
+				(font
+					(size 1.27 1.27)
+				)
+			)
+		)
+		(property "Datasheet" "https://www.tme.eu/Document/ca7ed7e840192927c2f50631891ac6c9/SP05xxBA.pdf"
+			(at 24.13 227.33 0)
+			(hide yes)
+			(show_name no)
+			(do_not_autoplace no)
+			(effects
+				(font
+					(size 1.27 1.27)
+				)
+			)
+		)
+		(property "Description" "SOT-143 TVS Diode array, 3xUnidirectional, 5.5V, Alternate KiCAD Library"
+			(at 24.13 227.33 0)
+			(hide yes)
+			(show_name no)
+			(do_not_autoplace no)
+			(effects
+				(font
+					(size 1.27 1.27)
+				)
+			)
+		)
+		(pin "1"
+		)
+		(pin "2"
+		)
+		(pin "4"
+		)
+		(pin "3"
+		)
+		(instances
+			(project "Mainboard layout"
+				(path "/322d2c9f-d9a6-40cc-b638-389f55be9478"
+					(reference "D2")
+					(unit 1)
+				)
