File: Hardware/KiCAD files/Mainboard layout/Mainboard layout Pre-16 pin SD module.kicad_pcb (KiCad board)
At the start: 2 copper layers, 191.3 x 169.2 mm, 80 parts, among them J10 Conn_01x02, J11 Conn_01x04, J12 JST_06, J13 Conn_01x08, J14 Conn_01x08, J17 PINHD_1x8_Male, J18 PINHD_1x8_Male, J19 PINHD_1x8_Male, J2 Screw_Terminal_2_P5.00mm, J20 PINHD_1x8_Male, J22 PINHD_1x8_Male, J23 PINHD_1x8_Male, J24 PINHD_1x8_Male, J25 Conn_01x04, J26 Conn_01x04, J27 Conn_01x04, J28 PINHD_1x8_Male, J3 Screw_Terminal_2_P3.50mm, J30 USB-A1VSB6, J31 JST_03, J32 USB-A1VSB6, J34 JST_03, J35 JST_03, J36 JST_03, J37 JST_03, J38 JST_03, J4 JST_06, J5 Conn_01x04, J6 JST_06, J7 JST_06, J8 Conn_01x06, J9 Conn_01x10, Q1 BS170, Q2 2DD1664, SW1 210-4MS, SW2 210-4MS, SW3 210-4MS, SW4 210-4MS, SW8 Push_Button, SW9 Push_Button, U1 CP2102-GM, U12 ESP32-S3-WROOM-1

Commit message: Most recent changes to final submission
Parts:
- removed J14: Conn_01x08, PCM_SparkFun-Connector:1x08_P2.54mm
- removed JP1, JP2: ~, PCM_SparkFun-Jumper:Jumper_2_NO
- added J1: MSD-1-A, Connector_Card:SD_Hirose_DM1AA_SF_PEJ82, F.Cu at (213.9, 97.3)
- added U3: PCA9534PW, PCM_SparkFun-Semiconductor-Standard:TSSOP-16_4.4x5mm_P0.65mm, F.Cu at (127.0, 33.9)
- added U5: PCA9534PW, PCM_SparkFun-Semiconductor-Standard:TSSOP-16_4.4x5mm_P0.65mm, F.Cu at (129.4, 47.0)
Routing:
- net GND: track 1451.5 -> 1426.8 mm
- net +3.3V: track 702.4 -> 695.8 mm, vias 31 -> 30
- net MOSI_1: track 78.8 -> 72.9 mm
- net SPI1_CS: track 230.1 -> 224.5 mm
- net SPI1_CLK: track 210.7 -> 205.8 mm
- net CHAINL0_MISO_1: track 132.3 -> 127.6 mm
- net /5V: track 3.00 -> 0.00 mm
- net +5V: track 262.4 -> 260.9 mm
