File: Hardware/KiCAD files/Mainboard layout/Mainboard layout.kicad_pcb (KiCad board)
At the start: 2 copper layers, 191.3 x 169.2 mm, 80 parts, among them J10 Conn_01x02, J11 Conn_01x04, J12 JST_06, J13 Conn_01x08, J14 Conn_01x08, J17 PINHD_1x8_Male, J18 PINHD_1x8_Male, J19 PINHD_1x8_Male, J2 Screw_Terminal_2_P5.00mm, J20 PINHD_1x8_Male, J22 PINHD_1x8_Male, J23 PINHD_1x8_Male, J24 PINHD_1x8_Male, J25 Conn_01x04, J26 Conn_01x04, J27 Conn_01x04, J28 PINHD_1x8_Male, J3 Screw_Terminal_2_P3.50mm, J30 USB-A1VSB6, J31 JST_03, J32 USB-A1VSB6, J34 JST_03, J35 JST_03, J36 JST_03, J37 JST_03, J38 JST_03, J4 JST_06, J5 Conn_01x04, J6 JST_06, J7 JST_06, J8 Conn_01x06, J9 Conn_01x10, Q1 BS170, Q2 2DD1664, SW1 210-4MS, SW2 210-4MS, SW3 210-4MS, SW4 210-4MS, SW8 Push_Button, SW9 Push_Button, U1 CP2102-GM, U12 ESP32-S3-WROOM-1

Commit message: Slight adjustments for EMI
trace changes primarily
Parts:
- added J15: Screw_Terminal_2_P5.00mm, TerminalBlock_Phoenix:TerminalBlock_Phoenix_PT-1,5-2-5.0-H_1x02_P5.00mm_Horizontal, F.Cu at (220.4, 90.5)
- added R9: 1k, Resistor_SMD:R_0805_2012Metric, F.Cu at (122.9, 72.3)
- added U2: PCA9534PW_118, PCA9534PW:SOP65P640X110-16N, F.Cu at (129.3, 46.9)
- added U4: PCA9534PW_118, PCA9534PW:SOP65P640X110-16N, F.Cu at (127.0, 33.9)
- C16: footprint PCM_SparkFun-Capacitor:C_0603_1608Metric -> LED_SMD:LED_0805_2012Metric
- C23: footprint PCM_SparkFun-Capacitor:C_0603_1608Metric -> Capacitor_SMD:C_0805_2012Metric
- R52, R53: footprint PCM_SparkFun-Resistor:R_0603_1608Metric -> LED_SMD:LED_0805_2012Metric
- R55, R56, R57: footprint PCM_SparkFun-Resistor:R_0603_1608Metric -> Resistor_SMD:R_0805_2012Metric
- moved R36 0.54 mm to (136.4, 29.0)
- moved R53 0.46 mm to (158.8, 31.2)
- moved R52 0.45 mm to (156.0, 30.0)
Connections:
- J28 pad 7: DRIVER_0_STEP -> DRIVER_E_STEP
- R107 pad 1: DRIVER_0_STEP -> DRIVER_E_STEP
- R50 pad 1: Step -> STEP
- U12 pad 4: Step -> STEP
Routing:
- net nSLP: track 240.8 -> 156.1 mm, vias 20 -> 12
- net DRIVER_0_STEP: track 265.9 -> 194.0 mm, vias 12 -> 10
- net +3.3V: track 702.4 -> 764.5 mm, vias 31 -> 32
- net DRIVER_E_STEP: track 0.00 -> 62.0 mm, vias 0 -> 2
- net STEPE: track 0.00 -> 41.2 mm, vias 0 -> 2
- net GND: track 1451.5 -> 1410.7 mm, vias 53 -> 78
- net STEP: track 0.00 -> 39.0 mm, vias 0 -> 2
- net IO_Interupter1: track 89.9 -> 68.4 mm, vias 8 -> 5
- net (no net): track 0.00 -> 13.3 mm, vias 0 -> 1
- net Step: track 8.82 -> 0.00 mm, vias 2 -> 0
- net CHAINL0_MISO_4: track 67.1 -> 59.3 mm
- net SPI4_CLK: track 212.8 -> 206.6 mm
- net *Suspend: track 126.1 -> 131.5 mm
- net N_ENBL: track 226.6 -> 223.2 mm
- net DATA_SELECT: track 160.9 -> 157.6 mm
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