File: Hardware/KiCAD files/Mainboard master/Peripherals.kicad_sch (KiCad schematic)
At the start: 33 parts, among them J3 Screw_Terminal_2_P3.50mm, J30 USB-A1VSB6, J31 JST_03, J34 JST_03, J35 JST_03, J36 JST_03, J37 JST_03, J38 JST_03, J39 JST_03, Q4 2N7000, U13 MAX31865, X1 3.5mm, X2 3.5mm

Commit message: another hotfix to the board, little adjustments
Other:
- moved on the sheet: J31, J34, OC1
Changed lines of the file:
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@@
 	(text "confirm fan wiring and connector on ender3\n\n"
 		(exclude_from_sim no)
-		(at 238.252 94.742 0)
+		(at 282.702 24.892 0)
 		(effects
 			(font
@@
 	)
 	(no_connect
-		(at 237.49 105.41)
+		(at 281.94 35.56)
 	)
 	(no_connect
-		(at 237.49 116.84)
+		(at 281.94 46.99)
 	)
 	(no_connect
@@
 	(polyline
 		(pts
-			(xy 244.475 178.435) (xy 244.475 262.255)
+			(xy 229.87 178.435) (xy 229.87 262.255)
 		)
 		(stroke
@@
 		)
 	)
+	(polyline
+		(pts
+			(xy 130.81 178.435) (xy 147.955 178.435)
+		)
+		(stroke
+			(width 0)
+			(type default)
+		)
+	)
 	(wire
 		(pts
@@
 	(polyline
 		(pts
-			(xy 244.475 262.255) (xy 13.335 262.255)
+			(xy 229.87 262.255) (xy 13.335 262.255)
 		)
 		(stroke
@@
 	(polyline
 		(pts
-			(xy 268.605 87.63) (xy 268.605 119.38)
+			(xy 313.055 17.78) (xy 313.055 49.53)
 		)
 		(stroke
@@
 	(polyline
 		(pts
-			(xy 80.01 91.44) (xy 147.32 91.44)
+			(xy 80.01 91.44) (xy 130.81 91.44)
 		)
 		(stroke
@@
 	(polyline
 		(pts
-			(xy 147.32 178.435) (xy 244.475 178.435)
+			(xy 147.32 178.435) (xy 229.87 178.435)
 		)
 		(stroke
@@
 	(polyline
 		(pts
-			(xy 210.185 88.265) (xy 268.605 88.265)
+			(xy 254.635 18.415) (xy 313.055 18.415)
 		)
 		(stroke
@@
 	(polyline
 		(pts
-			(xy 268.605 119.38) (xy 210.185 119.38)
+			(xy 313.055 49.53) (xy 254.635 49.53)
 		)
 		(stroke
@@
 	(wire
 		(pts
-			(xy 229.87 102.87) (xy 237.49 102.87)
+			(xy 274.32 33.02) (xy 281.94 33.02)
 		)
 		(stroke
@@
 	(polyline
 		(pts
-			(xy 147.32 91.44) (xy 147.32 178.435)
+			(xy 130.81 91.44) (xy 130.81 178.435)
 		)
 		(stroke
@@
 	(polyline
 		(pts
-			(xy 210.185 119.38) (xy 210.185 88.265)
+			(xy 254.635 49.53) (xy 254.635 18.415)
 		)
 		(stroke
@@
 	(polyline
 		(pts
-			(xy 268.605 88.265) (xy 268.605 88.9)
+			(xy 313.055 18.415) (xy 313.055 19.05)
 		)
 		(stroke
@@
 	(wire
 		(pts
-			(xy 229.87 114.3) (xy 237.49 114.3)
+			(xy 274.32 44.45) (xy 281.94 44.45)
 		)
 		(stroke
@@
 	(global_label "+3.3V"
 		(shape input)
-		(at 237.49 100.33 180)
+		(at 281.94 30.48 180)
 		(fields_autoplaced yes)
 		(effects
@@
 		)
 		(property "Intersheetrefs" "${INTERSHEET_REFS}"
-			(at 228.82 100.33 0)
+			(at 273.27 30.48 0)
 			(hide yes)
 			(show_name no)
@@
 	(global_label "+3.3V"
 		(shape input)
-		(at 237.49 111.76 180)
+		(at 281.94 41.91 180)
 		(fields_autoplaced yes)
 		(effects
@@
 		)
 		(property "Intersheetrefs" "${INTERSHEET_REFS}"
-			(at 228.82 111.76 0)
+			(at 273.27 41.91 0)
 			(hide yes)
 			(show_name no)
@@
 	(symbol
 		(lib_id "PCM_SparkFun-PowerSymbol:GND")
-		(at 229.87 102.87 270)
+		(at 274.32 33.02 270)
 		(unit 1)
 		(body_style 1)
@@
 		(fields_autoplaced yes)
 		(property "Reference" "#PWR021"
-			(at 223.52 102.87 0)
+			(at 267.97 33.02 0)
 			(hide yes)
 			(show_name no)
@@
 		)
 		(property "Value" "GND"
-			(at 226.06 102.87 0)
+			(at 270.51 33.02 0)
 			(show_name no)
 			(do_not_autoplace yes)
@@
 		)
 		(property "Footprint" ""
-			(at 229.87 102.87 0)
+			(at 274.32 33.02 0)
 			(hide yes)
 			(show_name no)
@@
 		)
 		(property "Datasheet" ""
-			(at 229.87 102.87 0)
+			(at 274.32 33.02 0)
 			(hide yes)
 			(show_name no)
@@
 		)
 		(property "Description" "Power symbol creates a global label with name \"GND\" , ground"
-			(at 220.98 102.87 0)
+			(at 265.43 33.02 0)
 			(hide yes)
 			(show_name no)
@@
 	(symbol
 		(lib_id "PCM_Optocoupler_Gate_Driver_AKL:ACNW3130")
-		(at 43.18 62.23 0)
+		(at 33.02 160.02 0)
 		(unit 1)
 		(body_style 1)
@@
 		(fields_autoplaced yes)
 		(property "Reference" "OC1"
-			(at 43.18 49.53 0)
+			(at 33.02 147.32 0)
 			(show_name no)
 			(do_not_autoplace no)
@@
 		)
 		(property "Value" "ACNW3130"
-			(at 43.18 52.07 0)
+			(at 33.02 149.86 0)
 			(show_name no)
 			(do_not_autoplace no)
@@
 		)
 		(property "Footprint" "PCM_Package_DIP_AKL:DIP-8_W7.62mm_LongPads"
-			(at 38.1 64.77 0)
+			(at 27.94 162.56 0)
 			(hide yes)
 			(show_name no)
@@
 		)
 		(property "Datasheet" "https://www.tme.eu/Document/8c4fd4552f89c48db87c694efad37ef3/ACNW3130-000E.pdf"
-			(at 40.64 62.23 0)
+			(at 30.48 160.02 0)
 			(hide yes)
 			(show_name no)
@@
 		)
 		(property "Description" "DIP-8 Optocoupler, Gate Driver output, 5kV, 2.5A, 100ns, Alternate KiCAD Library"
-			(at 43.18 62.23 0)
+			(at 33.02 160.02 0)
 			(hide yes)
 			(show_name no)
@@
 	(symbol
 		(lib_id "PCM_SparkFun-PowerSymbol:GND")
-		(at 229.87 114.3 270)
+		(at 274.32 44.45 270)
 		(unit 1)
 		(body_style 1)
@@
 		(fields_autoplaced yes)
 		(property "Reference" "#PWR020"
-			(at 223.52 114.3 0)
+			(at 267.97 44.45 0)
 			(hide yes)
 			(show_name no)
@@
 		)
 		(property "Value" "GND"
-			(at 226.06 114.3 0)
+			(at 270.51 44.45 0)
 			(show_name no)
 			(do_not_autoplace yes)
@@
 		)
 		(property "Footprint" ""
-			(at 229.87 114.3 0)
+			(at 274.32 44.45 0)
 			(hide yes)
 			(show_name no)
@@
 		)
 		(property "Datasheet" ""
-			(at 229.87 114.3 0)
+			(at 274.32 44.45 0)
 			(hide yes)
 			(show_name no)
@@
 		)
 		(property "Description" "Power symbol creates a global label with name \"GND\" , ground"
-			(at 220.98 114.3 0)
+			(at 265.43 44.45 0)
 			(hide yes)
 			(show_name no)
@@
 	(symbol
 		(lib_id "PCM_SL_Connectors:JST_03")
-		(at 241.3 114.3 0)
+		(at 285.75 44.45 0)
 		(unit 1)
 		(body_style 1)
@@
 		(fields_autoplaced yes)
 		(property "Reference" "J34"
-			(at 243.84 113.0299 0)
+			(at 288.29 43.1799 0)
 			(show_name no)
 			(do_not_autoplace no)
@@
 		)
 		(property "Value" "JST_03"
-			(at 243.84 115.5699 0)
+			(at 288.29 45.7199 0)
 			(show_name no)
 			(do_not_autoplace no)
@@
 		)
 		(property "Footprint" "Connector_JST:JST_EH_B3B-EH-A_1x03_P2.50mm_Vertical"
-			(at 241.3 106.68 0)
+			(at 285.75 36.83 0)
 			(hide yes)
 			(show_name no)
@@
 		)
 		(property "Datasheet" ""
-			(at 241.3 106.68 0)
+			(at 285.75 36.83 0)
 			(hide yes)
 			(show_name no)
@@
 		)
 		(property "Description" "JST Connector  3 pins"
-			(at 241.3 114.3 0)
+			(at 285.75 44.45 0)
 			(hide yes)
 			(show_name no)
@@
 	(symbol
 		(lib_id "PCM_SL_Connectors:JST_03")
-		(at 241.3 102.87 0)
+		(at 285.75 33.02 0)
 		(unit 1)
 		(body_style 1)
@@
 		(fields_autoplaced yes)
 		(property "Reference" "J31"
-			(at 243.84 101.5999 0)
+			(at 288.29 31.7499 0)
 			(show_name no)
 			(do_not_autoplace no)
@@
 		)
 		(property "Value" "JST_03"
-			(at 243.84 104.1399 0)
+			(at 288.29 34.2899 0)
 			(show_name no)
 			(do_not_autoplace no)
@@
 		)
 		(property "Footprint" "Connector_JST:JST_EH_B3B-EH-A_1x03_P2.50mm_Vertical"
-			(at 241.3 95.25 0)
+			(at 285.75 25.4 0)
 			(hide yes)
 			(show_name no)
@@
 		)
 		(property "Datasheet" ""
-			(at 241.3 95.25 0)
+			(at 285.75 25.4 0)
 			(hide yes)
 			(show_name no)
@@
 		)
 		(property "Description" "JST Connector  3 pins"
-			(at 241.3 102.87 0)
+			(at 285.75 33.02 0)
 			(hide yes)
 			(show_name no)

Commit message: general updates to the schematics and layouts
includes some backchecks tot he master schematic to be accurate for the paper
Parts:
- removed C1: 1nF_Ceramic, Capacitor_THT:C_Disc_D5.0mm_W2.5mm_P2.50mm, symbol PCM_SL_Capacitors:1nF_Ceramic
- removed J30: USB-A1VSB6, USB-A1VSB6:ONSHORE_USB-A1VSB6, symbol USB-A1VSB6:USB-A1VSB6
- removed R6: 1M, PCM_SparkFun-Resistor:R_0603_1608Metric, symbol PCM_SparkFun-Resistor:1M_0603
- added C16: 4.7uF, PCM_SparkFun-Capacitor:C_0603_1608Metric, symbol PCM_SparkFun-Capacitor:4.7uF_0603_35V_20%
- added C47, C67: 0.1uF, PCM_SparkFun-Capacitor:C_0603_1608Metric, symbol PCM_SparkFun-Capacitor:0.1uF_0603_25V_20%
- added C66: 1.0uF, PCM_SparkFun-Capacitor:C_0805_2012Metric, symbol PCM_SparkFun-Capacitor:1.0uF_0805_25V_10%
- added D14, D15: SP0503BAHT, PCM_Package_TO_SOT_SMD_AKL:SOT-143, symbol PCM_Diode_TVS_AKL:SP0503BAHT
- added D9: SP0502BAJT, PCM_Package_TO_SOT_SMD_AKL:SOT-323_SC-70, symbol PCM_Diode_TVS_AKL:SP0502BAJT
- added J1: MSD-1-A, Connector_Card:SD_Hirose_DM1AA_SF_PEJ82, symbol 2026-04-18_00-57-23:MSD-1-A
- added J32, J33: USB-A1VSB6, Connector_USB:USB_A_Kycon_KUSBX-AS1N-B_Horizontal, symbol USB-A1VSB6:USB-A1VSB6
- added R36, R48: 10k, Resistor_THT:R_Axial_DIN0207_L6.3mm_D2.5mm_P10.16mm_Horizontal, symbol PCM_SL_Resistors:10k
- added U3: CP2102-GM, CP2102:QFN28_5X5_SIL, symbol 2026-04-20_20-31-56:CP2102-GM
- renumbered ILI9341_MSP2202LCD1 to ILI9341_MSP2802LCD1
Connections:
- net +3.3V: now also C16.1, C47.1, J1.4 (VDD), U3.6 (VDD)
- net +5V: now also C66.1, C67.1, U3.7 (REGIN)
- net CHAINL0_MISO_1: now also J1.7 (DAT0)
- net GND: now also C16.2, C47.2, C66.2, C67.2, D14.1 (VN), D15.1 (VN), D9.3 (A), J1.6 (VSS), J32.4 (GND), J32.S1 (SHIELD), J32.S2 (SHIELD__1), J33.4 (GND), J33.S1 (SHIELD), J33.S2 (SHIELD__1), R36.1, R48.2, U3.29 (EPAD), U3.3 (GND)
- net MOSI_1: now also J1.3 (CMD)
- net SPI1_CLK: now also J1.5 (CLK)
- net SPI1_CS: now also J1.2 (CD/DAT3)
- new net *Suspend: R48.1, U3.11 (*SUSPEND)
- new net +5V_HIGHPW: D15.2 (L1), J33.1 (VUSB)
- new net CTS: U3.23 (CTS)
- new net DCD: U3.1 (DCD)
- new net DSR: U3.27 (DSR)
- new net DTR: U3.28 (DTR)
- new net PI_D+: D15.4 (L3), J33.3 (D+)
- new net PI_D-: D15.3 (L2), J33.2 (D-)
- new net Prog_D+: D14.4 (L3), J32.3 (D+), U3.4 (D+)
- new net Prog_D-: D14.3 (L2), J32.2 (D-), U3.5 (D-)
- new net RI: U3.2 (RI)
- new net RST: U3.9 (*RST)
- new net RTS: U3.24 (RTS)
- new net RX: D9.1 (K1), U3.25 (RXD)
- new net Suspend: R36.2, U3.12 (SUSPEND)
- new net TX: D9.2 (K2), U3.26 (TXD)
- new net VBus: D14.2 (L1), J32.1 (VUSB), U3.8 (VBUS)
- no-connect marks 7 -> 11
Other:
- note added: "CHECK FOOTPRINT FOR LARGER VERSION"
- note added: "Programmer_USB"
- note added: "RST - open drain output Regin - 5V in? CTS - Active low RTS - Active low DSR - Active Low DTR - Active Low DCD - Active Low RI - Active Low"
- note added: "TVS diode array or equivalent to SP0502BAHTG equivalent"
- note added: "USB_PI"
- note added: "Verify diodes"
- note removed: "USB"
