File: Hardware/KiCAD files/Mainbourd layout pre-weeks check 1/Mainboard Layout No daisy chain cp2102 moved/Mainboard Layout No daisy chain cp2102 moved.kicad_sch (KiCad schematic)
At the start: 93 parts, among them J1 JST_03, J11 Conn_01x04, J12 JST_06, J13 Conn_01x08, J14 Conn_01x08, J17 PINHD_1x8_Male, J18 PINHD_1x8_Male, J19 PINHD_1x8_Male, J2 Screw_Terminal_2_P5.00mm, J20 PINHD_1x8_Male, J22 PINHD_1x8_Male, J23 PINHD_1x8_Male, J24 PINHD_1x8_Male, J25 Conn_01x04, J26 Conn_01x04, J27 Conn_01x04, J28 PINHD_1x8_Male, J3 Screw_Terminal_2_P3.50mm, J30 USB-A1VSB6, J31 JST_03, J32 USB-A1VSB6, J34 JST_03, J35 JST_03, J36 JST_03, J37 JST_03, J38 JST_03, J4 JST_06, J5 Conn_01x04, J6 JST_06, J7 JST_06, J9 Conn_01x10, Q1 BS170, Q2 2DD1664, SW1 210-4MS, SW2 210-4MS, SW3 210-4MS, SW4 210-4MS, SW8 Push_Button, SW9 Push_Button, U1 CP2102-GM, U12 ESP32-S3-WROOM-1, U2 PCA9534PW_118, U4 PCA9534PW_118

Commit message: sick weekend changes
small adjustments left our some larger protection changes till after talking to weeks
Parts:
- removed JP1, JP2: (no value), PCM_SparkFun-Jumper:Jumper_2_NO, symbol PCM_SparkFun-Jumper:SolderJumper_2_Open
- added C17, C18, C19, C20: 10uF_1210_35V, Capacitor_SMD:C_1210_3225Metric, symbol PCM_4ms_Capacitor:10uF_1210_35V
- added D1: D_Generic, Diode_THT:D_DO-201AD_P15.24mm_Horizontal, symbol PCM_4ms_Diode:D_Generic
- added OC1, OC2, OC3: Optocoupler_Driver_Dual_Generic_Sep, symbol PCM_Optocoupler_Gate_Driver_AKL:Optocoupler_Driver_Dual_Generic_Sep
- added R15, R16: 0 ohmR_0805, PCM_Resistor_SMD_AKL:R_0805_2012Metric, symbol PCM_Resistor_AKL:R_0805
- added R17, R18: 0, Resistor_SMD:R_0805_2012Metric, symbol PCM_SL_Resistors:1k
- added TP1, TP2: TestPoint, TestPoint:TestPoint_Loop_D3.80mm_Drill2.5mm, symbol PCM_4ms_Connector:TestPoint
- added U3: ADuM1200ARZ, ADUM:R_8_ADI, symbol 2026-05-24_23-29-04:ADuM1200ARZ
- C1, C10, C11, C5: footprint PCM_SparkFun-Capacitor:Panasonic_D -> Capacitor_THT:C_Rect_L11.0mm_W3.5mm_P10.00mm_MKT; Voltage 25V -> 50V
- C2: value 10uF -> 22uF
- R1, R9: value 1k -> 0
Connections:
- net +24V: now also C1.1, C10.1, C11.1, C5.1, J17.1, J18.1, J19.1, J20.1
- net +5V: now also R18.1
- net +5V_HIGHPW: now also C19.1, D1.2 (A); no longer J32.1 (VUSB)
- net 3.3V: now also R17.2; no longer C16.1, C2.1, C23.1, C4.1, J13.3 (Pin_3), J26.1 (Pin_1), J31.1, J34.1, J35.3, J36.3, J37.3, J38.3, J5.1 (Pin_1), J9.1 (Pin_1), J9.8 (Pin_8), R12.1, R36.1, R41.2, R48.1, R49.2, R5.1, R50.2, R51.2, R52.2, R53.2, R55.1, R56.2, R57.1, SW1.1, SW1.2, SW1.3, SW1.4, SW2.1, SW2.2, SW2.3, SW2.4, SW3.1, SW3.2, SW3.3, SW3.4, SW4.1, SW4.2, SW4.3, SW4.4, U12.2 (3V3), U2.16 (VDD), U4.16 (VDD)
- net 5V: now also R18.2
- net GND: now also R41.2, C17.2, C18.2, C19.2, C20.2
- net PI_D+: now also R15.1; no longer U12.14 (GPIO20/U1CTS/ADC2_CH9/CLK_OUT1/USB_D+)
- net PI_D-: now also R16.1; no longer U12.13 (GPIO19/U1RTS/ADC2_CH8/CLK_OUT2/USB_D-)
- net at U12.5 (GPIO5/TOUCH5/ADC1_CH4): now also TP1.1
- net at U12.6 (GPIO6/TOUCH6/ADC1_CH5): now also TP2.1
- removed net +12V: C1.1, C10.1, C11.1, C5.1, J11.1 (Pin_1), J17.1, J18.1, J19.1, J20.1
- new net: D1.1 (K), J32.1 (VUSB)
- new net +3.3V: C16.1, C17.1, C18.1, C2.1, C23.1, C4.1, J13.3 (Pin_3), J26.1 (Pin_1), J31.1, J34.1, J35.3, J36.3, J37.3, J38.3, J5.1 (Pin_1), J9.1 (Pin_1), J9.8 (Pin_8), R12.1, R17.1, R36.1, R48.1, R49.2, R5.1, R50.2, R51.2, R52.2, R53.2, R55.1, R56.2, R57.1, SW1.1, SW1.2, SW1.3, SW1.4, SW2.1, SW2.2, SW2.3, SW2.4, SW3.1, SW3.2, SW3.3, SW3.4, SW4.1, SW4.2, SW4.3, SW4.4, U12.2 (3V3), U2.16 (VDD), U3.1 (VDD1), U4.16 (VDD)
- new net D+: R15.2, U12.14 (GPIO20/U1CTS/ADC2_CH9/CLK_OUT1/USB_D+)
- new net D-: R16.2, U12.13 (GPIO19/U1RTS/ADC2_CH8/CLK_OUT2/USB_D-)
- new net M+3.3V: C20.1, J11.1 (Pin_1), U3.8 (VDD2)
- no-connect marks 43 -> 42
Other:
- note added: "ISOLATION"
- note removed: "Pre-lim idea on muting backfeed onn 3.3V line"
- note removed: "TVS diode array or equivalent to SP0502BAHTG equivalent"
- note removed: "Verify diodes"
- note removed: "may want to have parralel interrupts"
- note removed: "verify that esp interrupt is on this pin"

Commit message: Compatability mods
basic modifications to work toward compatability between boards physically on the hotend
Parts:
- removed OC1, OC2, OC3: Optocoupler_Driver_Dual_Generic_Sep, symbol PCM_Optocoupler_Gate_Driver_AKL:Optocoupler_Driver_Dual_Generic_Sep
- added D2: D_Generic, Diode_THT:D_DO-201AD_P15.24mm_Horizontal, symbol PCM_4ms_Diode:D_Generic
Connections:
- net VBus: now also D2.2 (A); no longer J30.1 (VUSB)
- new net: D2.1 (K), J30.1 (VUSB)

Commit message: approved with final adjustments
Parts:
- added D3, D4: D_Generic, Diode_THT:D_DO-201AD_P15.24mm_Horizontal, symbol PCM_4ms_Diode:D_Generic
- J11, J25, J26, J27, J5: footprint PCM_SparkFun-Connector:1x04_P2.54mm -> PCM_SparkFun-Connector:1x03_P2.54mm; symbol PCM_SparkFun-Connector:Conn_01x04_P2.54mm -> PCM_SparkFun-Connector:Conn_01x03_P2.54mm
- R1: footprint Resistor_THT:R_Axial_DIN0207_L6.3mm_D2.5mm_P10.16mm_Horizontal -> Resistor_SMD:R_0805_2012Metric
Connections:
- net TX is gone; now on net RX: R8.2, U1.26 (TXD)
- net +5V: now also D3.2 (A); no longer J3.2
- net GND: no longer J11.4 (Pin_4), J25.4 (Pin_4), J26.4 (Pin_4), J27.4 (Pin_4), J5.4 (Pin_4)
- net SSR_Switch: now also D4.2 (A); no longer J3.1
- new net: D4.1 (K), J3.1
- new net: D3.1 (K), J3.2
Other:
- note added: "adc may read a bit lower than actual"

Commit message: V1 boards after final board invoice
Other:
- note added: "REGULATORS 3.3V, 5V"
- note removed: "REGULATORS 3.3V, 5V, 12V"
- moved on the sheet: J14, J31, J34, J35, J36, J37, J38, J9, R17, R18, U3
