File: Hardware/KiCAD files/LM2576_Var_Volt_Reg/LM2576_Var_Volt_Reg_12V.kicad_sch (KiCad schematic)
At the start: 13 parts, among them J1 Conn_01x03_Pin, U2 LM2576HVS-ADJ

Commit message: V2 mainboard
Parts:
- R1: value 2k -> 1k
- R4: value 19512 -> 8756
Changed lines of the file:
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@@
 		)
 		(instances
-			(project "LM2576_Var_Volt_Reg"
+			(project "LM2576_Var_Volt_Reg_12V"
 				(path "/05ad55a9-73a4-4419-8d6d-9b068d5aca56"
 					(reference "D2")
@@
 		)
 		(instances
-			(project "LM2576_Var_Volt_Reg"
+			(project "LM2576_Var_Volt_Reg_12V"
 				(path "/05ad55a9-73a4-4419-8d6d-9b068d5aca56"
 					(reference "#PWR05")
@@
 		)
 		(instances
-			(project "LM2576_Var_Volt_Reg"
+			(project "LM2576_Var_Volt_Reg_12V"
 				(path "/05ad55a9-73a4-4419-8d6d-9b068d5aca56"
 					(reference "#PWR08")
@@
 		)
 		(instances
-			(project "LM2576_Var_Volt_Reg"
+			(project "LM2576_Var_Volt_Reg_12V"
 				(path "/05ad55a9-73a4-4419-8d6d-9b068d5aca56"
 					(reference "#PWR01")
@@
 		)
 		(instances
-			(project "LM2576_Var_Volt_Reg"
+			(project "LM2576_Var_Volt_Reg_12V"
 				(path "/05ad55a9-73a4-4419-8d6d-9b068d5aca56"
 					(reference "L1")
@@
 			)
 		)
-		(property "Value" "19512"
+		(property "Value" "8756"
 			(at 165.1 81.2799 0)
 			(show_name no)
@@
 		)
 		(instances
-			(project "LM2576_Var_Volt_Reg"
+			(project "LM2576_Var_Volt_Reg_12V"
 				(path "/05ad55a9-73a4-4419-8d6d-9b068d5aca56"
 					(reference "R4")
@@
 		)
 		(instances
-			(project "LM2576_Var_Volt_Reg"
+			(project "LM2576_Var_Volt_Reg_12V"
 				(path "/05ad55a9-73a4-4419-8d6d-9b068d5aca56"
 					(reference "#PWR07")
@@
 		)
 		(instances
-			(project "LM2576_Var_Volt_Reg"
+			(project "LM2576_Var_Volt_Reg_12V"
 				(path "/05ad55a9-73a4-4419-8d6d-9b068d5aca56"
 					(reference "#PWR03")
@@
 			)
 		)
-		(property "Value" "2k"
+		(property "Value" "1k"
 			(at 165.1 91.4399 0)
 			(show_name no)
@@
 		)
 		(instances
-			(project "LM2576_Var_Volt_Reg"
+			(project "LM2576_Var_Volt_Reg_12V"
 				(path "/05ad55a9-73a4-4419-8d6d-9b068d5aca56"
 					(reference "R1")
@@
 		)
 		(instances
-			(project "LM2576_Var_Volt_Reg"
+			(project "LM2576_Var_Volt_Reg_12V"
 				(path "/05ad55a9-73a4-4419-8d6d-9b068d5aca56"
 					(reference "#PWR04")
@@
 		)
 		(instances
-			(project "LM2576_Var_Volt_Reg"
+			(project "LM2576_Var_Volt_Reg_12V"
 				(path "/05ad55a9-73a4-4419-8d6d-9b068d5aca56"
 					(reference "C1")
@@
 		)
 		(instances
-			(project "LM2576_Var_Volt_Reg"
+			(project "LM2576_Var_Volt_Reg_12V"
 				(path "/05ad55a9-73a4-4419-8d6d-9b068d5aca56"
 					(reference "C3")
@@
 		)
 		(instances
-			(project "LM2576_Var_Volt_Reg"
+			(project "LM2576_Var_Volt_Reg_12V"
 				(path "/05ad55a9-73a4-4419-8d6d-9b068d5aca56"
 					(reference "C5")
@@
 		)
 		(instances
-			(project "LM2576_Var_Volt_Reg"
+			(project "LM2576_Var_Volt_Reg_12V"
 				(path "/05ad55a9-73a4-4419-8d6d-9b068d5aca56"
 					(reference "#PWR02")
@@
 		)
 		(instances
-			(project "LM2576_Var_Volt_Reg"
+			(project "LM2576_Var_Volt_Reg_12V"
 				(path "/05ad55a9-73a4-4419-8d6d-9b068d5aca56"
 					(reference "U2")
@@
 		)
 		(instances
-			(project "LM2576_Var_Volt_Reg"
+			(project "LM2576_Var_Volt_Reg_12V"
 				(path "/05ad55a9-73a4-4419-8d6d-9b068d5aca56"
 					(reference "J1")
@@
 		)
 		(instances
-			(project "LM2576_Var_Volt_Reg"
+			(project "LM2576_Var_Volt_Reg_12V"
 				(path "/05ad55a9-73a4-4419-8d6d-9b068d5aca56"
 					(reference "#PWR06")
@@
 		)
 		(instances
-			(project "LM2576_Var_Volt_Reg"
+			(project "LM2576_Var_Volt_Reg_12V"
 				(path "/05ad55a9-73a4-4419-8d6d-9b068d5aca56"
 					(reference "C2")
@@
 		)
 		(instances
-			(project "LM2576_Var_Volt_Reg"
+			(project "LM2576_Var_Volt_Reg_12V"
 				(path "/05ad55a9-73a4-4419-8d6d-9b068d5aca56"
 					(reference "R3")
@@
 		)
 		(instances
-			(project "LM2576_Var_Volt_Reg"
+			(project "LM2576_Var_Volt_Reg_12V"
 				(path "/05ad55a9-73a4-4419-8d6d-9b068d5aca56"
 					(reference "C4")
@@
 		)
 		(instances
-			(project "LM2576_Var_Volt_Reg"
+			(project "LM2576_Var_Volt_Reg_12V"
 				(path "/05ad55a9-73a4-4419-8d6d-9b068d5aca56"
 					(reference "CR2")
