File: Hardware/KiCAD files/Mainbourd layout pre-weeks check 1/V2 checks/Mainboard V2.kicad_sch (KiCad schematic)
At the start: 106 parts, among them J1 JST_03, J11 Conn_01x04, J12 JST_06, J13 Conn_01x08, J14 Conn_01x08, J17 PINHD_1x8_Male, J18 PINHD_1x8_Male, J19 PINHD_1x8_Male, J2 Screw_Terminal_2_P5.00mm, J20 PINHD_1x8_Male, J22 PINHD_1x8_Male, J23 PINHD_1x8_Male, J24 PINHD_1x8_Male, J25 Conn_01x04, J26 Conn_01x04, J27 Conn_01x04, J28 PINHD_1x8_Male, J3 Screw_Terminal_2_P3.50mm, J30 USB-A1VSB6, J31 JST_03, J32 USB-A1VSB6, J34 JST_03, J35 JST_03, J36 JST_03, J37 JST_03, J38 JST_03, J4 JST_06, J5 Conn_01x04, J6 JST_06, J7 JST_06, J9 Conn_01x10, Q1 BS170, Q2 2DD1664, SW1 210-4MS, SW2 210-4MS, SW3 210-4MS, SW4 210-4MS, SW8 Push_Button, SW9 Push_Button, U1 CP2102-GM, U12 ESP32-S3-WROOM-1, U2 PCA9534PW_118, U3 ADuM1200ARZ, U4 PCA9534PW_118

Commit message: V2 mainboard
Parts:
- removed C16: 0.1uF, LED_SMD:LED_0805_2012Metric, symbol PCM_SparkFun-Capacitor:0.1uF_0603_25V_20%
- removed C23: 0.1uF, Capacitor_SMD:C_0805_2012Metric, symbol PCM_SparkFun-Capacitor:0.1uF_0603_25V_20%
- removed D1: D_Generic, Diode_THT:D_DO-201AD_P15.24mm_Horizontal, symbol PCM_4ms_Diode:D_Generic
- removed J14: Conn_01x08, PCM_SparkFun-Connector:1x08_P2.54mm, symbol PCM_SparkFun-Connector:Conn_01x08_P2.54mm
- removed J31, J34: JST_03, Connector_JST:JST_EH_B3B-EH-A_1x03_P2.50mm_Vertical, symbol PCM_SL_Connectors:JST_03
- removed J9: Conn_01x10, PCM_SparkFun-Connector:1x10_P2.54mm, symbol PCM_SparkFun-Connector:Conn_01x10_P2.54mm
- removed R1, R17, R18, R9: 0, Resistor_SMD:R_0805_2012Metric, symbol PCM_SL_Resistors:1k
- removed R107, R89, R90, R91: 4K7, PCM_SparkFun-Resistor:R_0603_1608Metric, symbol Device:R_Small
- removed R11, R3: 100, Resistor_SMD:R_0805_2012Metric, symbol PCM_SparkFun-Resistor:100_0603
- removed R49, R51, R56, R57: 10k, Resistor_SMD:R_0805_2012Metric, symbol PCM_SparkFun-Resistor:10k_0603
- removed R50: 1k, Resistor_THT:R_Axial_DIN0207_L6.3mm_D2.5mm_P10.16mm_Horizontal, symbol PCM_SparkFun-Resistor:10k_0603
- removed R6: 10k, Resistor_THT:R_Axial_DIN0207_L6.3mm_D2.5mm_P10.16mm_Horizontal, symbol PCM_SL_Resistors:10k
- removed U2, U4: PCA9534PW_118, PCA9534PW:SOP65P640X110-16N, symbol PCA9534PW_118:PCA9534PW_118
- added J10, J8: JST_02, Connector_JST:JST_EH_B2B-EH-A_1x02_P2.50mm_Vertical, symbol PCM_SL_Connectors:JST_02
- added J14: Conn_01x10, PCM_SparkFun-Connector:1x10_P2.54mm, symbol PCM_SparkFun-Connector:Conn_01x10_P2.54mm
- added J16: Conn_01x04, PCM_SparkFun-Connector:1x04_P2.54mm, symbol PCM_SparkFun-Connector:Conn_01x04_P2.54mm
- added J9: Conn_01x08, PCM_SparkFun-Connector:1x08_P2.54mm, symbol PCM_SparkFun-Connector:Conn_01x08_P2.54mm
- added Q3: 2DD1664, PCM_Package_TO_SOT_SMD_AKL:SOT-89-3, symbol PCM_Transistor_BJT_AKL:2DD1664
- added R1: Resistor, Resistor_THT:R_Axial_DIN0207_L6.3mm_D2.5mm_P10.16mm_Horizontal, symbol PCM_SL_Devices:Resistor
- added R11, R17, R18, R19: 0 ohmR_0805, PCM_Resistor_SMD_AKL:R_0805_2012Metric, symbol PCM_Resistor_AKL:R_0805
- added U5: TCA9535PWR, PW0024A_N, symbol 2026-06-19_18-44-44:TCA9535PWR
- D2: footprint Diode_THT:D_DO-201AD_P15.24mm_Horizontal -> (none)
- TP1, TP2: footprint TestPoint:TestPoint_Loop_D3.80mm_Drill2.5mm -> TestPoint:TestPoint_Loop_D2.54mm_Drill1.5mm_Beaded
Connections:
- net DATA_SELECT is gone; now on an unnamed net: U12.23 (GPIO21)
- net DRIVER_E_STEP is gone; now on net STEPE: J28.7
- net *Suspend: no longer U1.11 (*SUSPEND)
- net +24V: now also J35.3, J36.3, J37.3, J38.3, Q3.2 (C)
- net +3.3V: now also J13.1 (Pin_1), J22.5, J22.6, J23.5, J23.6, J24.5, J24.6, J28.5, J28.6, J14.7 (Pin_7), J16.4 (Pin_4), J9.1 (Pin_1), U5.24 (VCC); no longer J13.3 (Pin_3), J35.3, J36.3, J37.3, J38.3
- net +5V_HIGHPW: now also J32.1 (VUSB)
- net AXIS_E_ENDSTOP: now also U5.10 (P06)
- net AXIS_X_ENDSTOP: now also U5.7 (P03)
- net AXIS_Y_ENDSTOP: now also U5.8 (P04)
- net AXIS_Z_ENDSTOP: now also U5.9 (P05)
- net D+: now also R15.1, TP1.1
- net D-: now also R16.1, TP2.1
- net DIR0: now also U5.17 (P14)
- net DIR1: now also U5.18 (P15)
- net DIR2: now also U5.19 (P16)
- net DIRE: now also U5.20 (P17)
- net GND: now also J10.2, J16.3 (Pin_3), J8.2, J9.2 (Pin_2), R1.2, U5.12 (GND), U5.2 (A1), U5.21 (A0), U5.3 (A2)
- net IO_Interupter1: now also U12.24 (GPIO47/SPICLK_P/SUBSPICLK_P_DIFF), U5.1 (INT_N); no longer U12.38 (GPIO2/TOUCH2/ADC1_CH1)
- net LCD_RESET: now also J16.1 (Pin_1)
- net MODE_0_GPIO0: now also J23.2, SW3.6; no longer J23.4, SW3.8
- net MODE_0_GPIO1: now also J22.2, SW2.6; no longer J22.4, SW2.8
- net MODE_0_GPIO2: now also J24.2, SW4.6; no longer J24.4, SW4.8
- net MODE_0_GPIOE: now also J28.2, SW1.6; no longer J28.4, SW1.8
- net MODE_2_GPIO0: now also J23.4, SW3.8; no longer J23.2, SW3.6
- net MODE_2_GPIO1: now also J22.4, SW2.8; no longer J22.2, SW2.6
- net MODE_2_GPIO2: now also J24.4, SW4.8; no longer J24.2, SW4.6
- net MODE_2_GPIOE: now also J28.4, SW1.8; no longer J28.2, SW1.6
- net Prog_D+: now also R11.2; no longer U1.4 (D+)
- net Prog_D-: now also R17.2; no longer U1.5 (D-)
- net Reset: no longer J22.5, J23.5, J24.5, J28.5, U12.39 (GPIO1/TOUCH1/ADC1_CH0)
- net STEPE: now also U12.7 (GPIO7/TOUCH7/ADC1_CH6)
- net Suspend: no longer U1.12 (SUSPEND)
- net VBus: now also J30.1 (VUSB); no longer D2.2 (A)
- net nSLP: no longer J22.6, J23.6, J24.6, J28.6
- net STEPZ: now reaches U12.6 (GPIO6/TOUCH6/ADC1_CH5)
- net STEPZ: now also J24.7; no longer TP2.1
- net at U12.11 (GPIO18/U1RXD/ADC2_CH7/CLK_OUT3): now also R19.2
- net at R7.1: now also U5.22 (SCL)
- net at R2.1: now also U5.23 (SDA)
- net at D2.1 (K): now also R1.1; no longer J30.1 (VUSB)
- net STEPY: now reaches U12.5 (GPIO5/TOUCH5/ADC1_CH4)
- net STEPY: now also J22.7; no longer TP1.1
- net at Q2.1 (B): no longer U12.31 (GPIO38/FSPIWP/SUBSPIWP)
- net TOUCHCS: now reaches U12.12 (GPIO8/TOUCH8/ADC1_CH7/SUBSPICS1)
- net TOUCHCS: now also J14.4 (Pin_4)
- net DC: now reaches U12.17 (GPIO9/TOUCH9/ADC1_CH8/FSPIHD/SUBSPIHD)
- net DC: now also J14.10 (Pin_10); no longer J1.2
- net at U12.25 (GPIO48/SPICLK_N/SUBSPICLK_N_DIFF): now also D2.2 (A)
- net DATA1: now reaches U12.33 (MTDO/GPIO40/CLK_OUT2)
- net DATA1: now also J9.8 (Pin_8)
- net DATA3: now reaches U12.35 (MTMS/GPIO42)
- net DATA3: now also J9.6 (Pin_6)
- net HeadIO1: now reaches J1.1
- net HeadIO1: now also U5.4 (P00); no longer U12.7 (GPIO7/TOUCH7/ADC1_CH6)
- net SDA: now reaches R2.2, R53.1
- net SDA: now also U12.39 (GPIO1/TOUCH1/ADC1_CH0); no longer U12.8 (GPIO15/U0RTS/ADC2_CH4/XTAL_32K_P)
- net SCL: now reaches R52.1, R7.2
- net SCL: now also U12.38 (GPIO2/TOUCH2/ADC1_CH1); no longer U12.9 (GPIO16/U0CTS/ADC2_CH5/XTAL_32K_N)
- net 3.3V_in1 renamed SSRE
- net SSRE: now also U5.6 (P02)
- net DRDY_ALOW: no longer names the net of J13.8 (Pin_8)
- net DRDY_ALOW: no longer U12.34 (MTDI/GPIO41/CLK_OUT1)
- removed net DRIVER_0_STEP: J22.7, J23.7, J24.7
- net IO_Interupter2 renamed DATA0
- net DATA0: now also J9.3 (Pin_3)
- net MISO_1 renamed MOSI
- net MOSI: now also J13.6 (Pin_6), J14.3 (Pin_3), J14.9 (Pin_9); no longer J13.7 (Pin_7)
- net MOSI_1 renamed MISO
- net MISO: now also J14.2 (Pin_2), J14.6 (Pin_6)
- removed net N_ENBL: J22.1, J23.1, J24.1, U12.26 (GPIO45)
- net N_ENBLE: no longer names the net of U12.16 (GPIO46)
- net N_ENBLE: no longer J28.1
- net PI_D+ renamed PI_TX
- net PI_TX: now also R18.1; no longer R15.1
- net PI_D- renamed PI_RX
- net PI_RX: now also R19.1; no longer R16.1
- net SPI1_1SS renamed CMD
- net CMD: now also J9.4 (Pin_4); no longer J13.6 (Pin_6)
- net SPI1_CLK renamed SPI_CLK
- net SPI_CLK: now also J14.5 (Pin_5), J14.8 (Pin_8)
- net SPI4_CLK: no longer names the net of U12.10 (GPIO17/U1TXD/ADC2_CH6)
- net SPI4_CLK: now also R18.2
- net STEP renamed STEPX
- net STEPX: now also J23.7
- new net: J10.1, J8.1, Q3.3 (E)
- new net DATA2: J9.7 (Pin_7), U12.34 (MTDI/GPIO41/CLK_OUT1)
- new net EEN: J28.1, U5.16 (P13)
- new net FAN_CTRL: Q3.1 (B), U5.11 (P07)
- new net HeadIO2: J1.2, U5.5 (P01)
- new net LCDCS: J16.2 (Pin_2), U12.8 (GPIO15/U0RTS/ADC2_CH4/XTAL_32K_P)
- new net PD+: R11.1, U1.4 (D+)
- new net PD-: R17.1, U1.5 (D-)
- new net RTDCS: J13.7 (Pin_7), U12.9 (GPIO16/U0CTS/ADC2_CH5/XTAL_32K_N)
- new net SD_CLK: J9.5 (Pin_5), U12.31 (GPIO38/FSPIWP/SUBSPIWP)
- new net TOUCH_INT: J14.1 (Pin_1)
- new net XEN: J23.1, U5.13 (P10)
- new net YEN: J22.1, U5.14 (P11)
- new net ZEN: J24.1, U5.15 (P12)
- no-connect marks 42 -> 39
Other:
- note added: "CHECK IF THERES NO SPARES CONNECTIONS FOR RESET AND NSLP"
- note added: "CUT SUSPEND TRACES TO TEST NECESITY"
- note added: "IO expander"
- note added: "SD MMC CARD"
- note added: "confirm fan wiring and connector on ender3 verify with ender 3 fans"
- note added: "confirm which of these connections are 2 pin or 3 pin on the mainboard"
- note added: "look into addding a resistor to ground"
- note removed: "DRV Step Pulldowns"
- note removed: "IO expanders"
- note removed: "SD CARD"
- note removed: "SPI is 1110"
- note removed: "STEP DISPERSAL"
- note removed: "adc may read a bit lower than actual"
- note removed: "confirm fan wiring and connector on ender3"
- note removed: "parrallel to the drivers"
- moved on the sheet: C15, J1, R2, R52, R53, R55, R7
