File: Hardware/KiCAD files/Mainbourd layout pre-weeks check 1/V2 checks/_restore_backup_2026-05-20T16-31-20-836/Mainboard Layout No daisy chain cp2102 moved.kicad_sch (KiCad schematic)
At the start: 106 parts, among them J1 JST_03, J11 Conn_01x04, J12 JST_06, J13 Conn_01x08, J14 Conn_01x08, J17 PINHD_1x8_Male, J18 PINHD_1x8_Male, J19 PINHD_1x8_Male, J2 Screw_Terminal_2_P5.00mm, J20 PINHD_1x8_Male, J22 PINHD_1x8_Male, J23 PINHD_1x8_Male, J24 PINHD_1x8_Male, J25 Conn_01x04, J26 Conn_01x04, J27 Conn_01x04, J28 PINHD_1x8_Male, J3 Screw_Terminal_2_P3.50mm, J30 USB-A1VSB6, J31 JST_03, J32 USB-A1VSB6, J34 JST_03, J35 JST_03, J36 JST_03, J37 JST_03, J38 JST_03, J4 JST_06, J5 Conn_01x04, J6 JST_06, J7 JST_06, J9 Conn_01x10, Q1 BS170, Q2 2DD1664, SW1 210-4MS, SW2 210-4MS, SW3 210-4MS, SW4 210-4MS, SW8 Push_Button, SW9 Push_Button, U1 CP2102-GM, U12 ESP32-S3-WROOM-1, U2 PCA9534PW_118, U3 ADuM1200ARZ, U4 PCA9534PW_118

Commit message: V2 mainboard
Parts:
- removed C12, C14: 1 uF, PCM_SparkFun-Capacitor:C_1210_3225Metric, symbol PCM_SparkFun-Capacitor:10uF_1210_50V_20%
- removed C13: .1 uF, PCM_SparkFun-Capacitor:C_1210_3225Metric, symbol PCM_SparkFun-Capacitor:10uF_1210_50V_20%
- removed C15: 0.1uF, Capacitor_SMD:C_0805_2012Metric, symbol PCM_SparkFun-Capacitor:0.1uF_0603_25V_20%
- removed C17, C18, C19, C20: 10uF_1210_35V, Capacitor_SMD:C_1210_3225Metric, symbol PCM_4ms_Capacitor:10uF_1210_35V
- removed D1, D2, D3, D4: D_Generic, Diode_THT:D_DO-201AD_P15.24mm_Horizontal, symbol PCM_4ms_Diode:D_Generic
- removed R10, R11: 100, Resistor_SMD:R_0805_2012Metric, symbol PCM_SparkFun-Resistor:100_0603
- removed R12: 10k, Resistor_THT:R_Axial_DIN0207_L6.3mm_D2.5mm_P10.16mm_Horizontal, symbol PCM_SL_Resistors:10k
- removed R13: 4.7k, Resistor_THT:R_Axial_DIN0207_L6.3mm_D2.5mm_P10.16mm_Horizontal, symbol PCM_SL_Resistors:10k
- removed R14, R15, R16, R8: 0 ohmR_0805, PCM_Resistor_SMD_AKL:R_0805_2012Metric, symbol PCM_Resistor_AKL:R_0805
- removed R17, R18: 0, Resistor_SMD:R_0805_2012Metric, symbol PCM_SL_Resistors:1k
- removed R51: 10k, Resistor_SMD:R_0805_2012Metric, symbol PCM_SparkFun-Resistor:10k_0603
- removed TP1, TP2: TestPoint, TestPoint:TestPoint_Loop_D3.80mm_Drill2.5mm, symbol PCM_4ms_Connector:TestPoint
- removed U3: ADuM1200ARZ, ADUM:R_8_ADI, symbol 2026-05-24_23-29-04:ADuM1200ARZ
- added D1: SP0502BAJT, PCM_Package_TO_SOT_SMD_AKL:SOT-323_SC-70, symbol PCM_Diode_TVS_AKL:SP0502BAJT
- added D10, D11, D2, D3: SP0503BAHT, PCM_Package_TO_SOT_SMD_AKL:SOT-143, symbol PCM_Diode_TVS_AKL:SP0503BAHT
- added J15: Screw_Terminal_2_P5.00mm, TerminalBlock_Phoenix:TerminalBlock_Phoenix_PT-1,5-2-5.0-H_1x02_P5.00mm_Horizontal, symbol PCM_SL_Screw_Terminal:Screw_Terminal_2_P5.00mm
- added JP1, JP2: (no value), PCM_SparkFun-Jumper:Jumper_2_NO, symbol PCM_SparkFun-Jumper:SolderJumper_2_Open
- added R8: 10k, Resistor_THT:R_Axial_DIN0207_L6.3mm_D2.5mm_P10.16mm_Horizontal, symbol PCM_SL_Resistors:10k
- C1, C10, C11, C5: footprint Capacitor_THT:C_Rect_L11.0mm_W3.5mm_P10.00mm_MKT -> PCM_SparkFun-Capacitor:Panasonic_D; Voltage 50V -> 25V
- C2: value 22uF -> 10uF
- C4: value .1 uF -> 10uF
- J11, J25, J26, J27, J5: footprint PCM_SparkFun-Connector:1x03_P2.54mm -> PCM_SparkFun-Connector:1x04_P2.54mm; symbol PCM_SparkFun-Connector:Conn_01x03_P2.54mm -> PCM_SparkFun-Connector:Conn_01x04_P2.54mm
- R1: value 0 -> 1k; footprint Resistor_SMD:R_0805_2012Metric -> Resistor_THT:R_Axial_DIN0207_L6.3mm_D2.5mm_P10.16mm_Horizontal
- R2: value 100 ohmR_0805 -> 50 ohmR_0805
- R7: value 100 ohm R_0805 -> 50 ohm R_0805
- R9: value 0 -> 1k
Connections:
- net D+ is gone; now on net PI_D+: U12.14 (GPIO20/U1CTS/ADC2_CH9/CLK_OUT1/USB_D+)
- net D- is gone; now on net PI_D-: U12.13 (GPIO19/U1RTS/ADC2_CH8/CLK_OUT2/USB_D-)
- net VDD is gone; now on net 3.3V: C6.1, C9.1, U1.6 (VDD)
- net +24V: no longer C1.1, C10.1, C11.1, C5.1, J17.1, J18.1, J19.1, J20.1
- net +5V: now also C7.1, C8.1, J3.2, U1.7 (REGIN), JP2.1 (A)
- net +5V_HIGHPW: now also J32.1 (VUSB), D11.2 (L1)
- net 3.3V: now also C16.1, C2.1, C23.1, J13.3 (Pin_3), J26.1 (Pin_1), J31.1, J34.1, J35.3, J36.3, J37.3, J38.3, J5.1 (Pin_1), J9.1 (Pin_1), J9.8 (Pin_8), R36.1, R41.2, R48.1, R49.2, R5.1, R50.2, R52.2, R53.2, R55.1, R56.2, R57.1, SW1.1, SW1.2, SW1.3, SW1.4, SW2.1, SW2.2, SW2.3, SW2.4, SW3.1, SW3.2, SW3.3, SW3.4, SW4.1, SW4.2, SW4.3, SW4.4, U12.2 (3V3), U2.16 (VDD), U4.16 (VDD), JP1.1 (A), JP1.2 (B)
- net 5V: now also JP2.2 (B)
- net GND: now also J11.4 (Pin_4), J25.4 (Pin_4), J26.4 (Pin_4), J27.4 (Pin_4), J5.4 (Pin_4), D1.3 (A), D10.1 (VN), D11.1 (VN), R8.1; no longer R41.2, SW8.2
- net MOSI_1: now also U12.21 (GPIO13/TOUCH13/ADC2_CH2/FSPIQ/FSPIIO7/SUBSPIQ)
- net MOSI_4: now also U12.11 (GPIO18/U1RXD/ADC2_CH7/CLK_OUT3)
- net N_ENBL: now also J28.1
- net PI_D+: now also D11.4 (L3)
- net PI_D-: now also D11.3 (L2)
- net Prog_D+: now also D10.4 (L3)
- net Prog_D-: now also D10.3 (L2)
- net RX: now also U12.36 (U0RXD/GPIO44/CLK_OUT2), D1.1 (K1); no longer U1.26 (TXD)
- net SPI4_1SS: now also U12.12 (GPIO8/TOUCH8/ADC1_CH7/SUBSPICS1); no longer U2.12 (IO7)
- net SSR_Switch: now also J3.1
- net Suspend: now also R8.2
- net VBus: now also J30.1 (VUSB), D10.2 (L1); no longer C7.1, C8.1, U1.7 (REGIN)
- net DCD: now reaches U12.6 (GPIO6/TOUCH6/ADC1_CH5)
- net DCD: now also U1.1 (DCD)
- net at SW8.1, U12.3 (EN): now also C4.1; no longer R5.2
- net at R7.1, U2.14 (SCL), U4.14 (SCL): now also R52.1
- net at R2.1, U2.15 (SDA), U4.15 (SDA): now also R53.1
- net RI: now reaches U1.2 (RI)
- net RI: now also U12.5 (GPIO5/TOUCH5/ADC1_CH4)
- net CTS: now reaches U1.23 (CTS)
- net CTS: now also U12.16 (GPIO46)
- net RTS: now reaches U1.24 (RTS)
- net RTS: now also U12.15 (GPIO3/TOUCH3/ADC1_CH2)
- net DSR: now reaches U1.27 (DSR)
- net DSR: now also U12.33 (MTDO/GPIO40/CLK_OUT2)
- net DTR: now reaches U1.28 (DTR)
- net DTR: now also U12.24 (GPIO47/SPICLK_P/SUBSPICLK_P_DIFF)
- net RST: now reaches U1.9 (*RST)
- net RST: now also U12.25 (GPIO48/SPICLK_N/SUBSPICLK_N_DIFF)
- net TX: now reaches U12.37 (U0TXD/GPIO43/CLK_OUT1)
- net TX: now also U1.26 (TXD), D1.2 (K2)
- net at R2.2, U12.8 (GPIO15/U0RTS/ADC2_CH4/XTAL_32K_P): no longer R53.1
- net at R7.2, U12.9 (GPIO16/U0CTS/ADC2_CH5/XTAL_32K_N): no longer R52.1
- net SPI4_0SS: now reaches U4.12 (IO7)
- removed net +3.3V: C16.1, C2.1, C23.1, C4.1, J13.3 (Pin_3), J26.1 (Pin_1), J31.1, J34.1, J35.3, J36.3, J37.3, J38.3, J5.1 (Pin_1), J9.1 (Pin_1), J9.8 (Pin_8), R36.1, R48.1, R49.2, R5.1, R50.2, R52.2, R53.2, R55.1, R56.2, R57.1, SW1.1, SW1.2, SW1.3, SW1.4, SW2.1, SW2.2, SW2.3, SW2.4, SW3.1, SW3.2, SW3.3, SW3.4, SW4.1, SW4.2, SW4.3, SW4.4, U12.2 (3V3), U2.16 (VDD), U4.16 (VDD)
- net M+3.3V renamed +12V
- net +12V: now also C1.1, C10.1, C11.1, C5.1, J17.1, J18.1, J19.1, J20.1
- removed net N_ENBLE: J28.1, U12.16 (GPIO46)
- new net: R5.2, SW8.2
- no-connect marks 42 -> 32
Other:
- note added: "IN CASE FOR SHIELDING"
- note added: "Pre-lim idea on muting backfeed onn 3.3V line"
- note added: "REGULATORS 3.3V, 5V, 12V"
- note added: "RST - open drain output Regin - 5V in? CTS - Active low RTS - Active low DSR - Active Low DTR - Active Low DCD - Active Low RI - Active Low"
- note added: "TVS diode array or equivalent to SP0502BAHTG equivalent"
- note added: "Verify diodes"
- note added: "may want to have parralel interrupts"
- note added: "verify that esp interrupt is on this pin"
- note removed: "IO expanders"
- note removed: "ISOLATION"
- note removed: "LEAVE R51 AND R49 EMPTY ONLY FOR TESTING"
- note removed: "REGULATORS 3.3V, 5V"
- note removed: "adc may read a bit lower than actual"
- note removed: "check C15"
- moved on the sheet: C2, C23, J14, J31, J34, J35, J36, J37, J38, J9, R2, R52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
